File: pcb/NFC2USB.kicad_sch (KiCad schematic)
At the start: 12 parts, among them J1 USB_C_Receptacle_USB2.0, U1 NFCModuleRC522, U2 AMS1117-3.3

Commit message: fix: add PWR_FLAGs
Changed lines of the file:
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@@
     (pin "2")
+  )
+  (symbol (lib_id "power:VBUS") (at -39.37 182.88 180) (unit 1)
+    (in_bom yes) (on_board yes) (fields_autoplaced)
+    (property "Reference" "#PWR?" (id 0) (at -39.37 179.07 0)
+      (effects (font (size 1.27 1.27)) hide)
+    )
+    (property "Value" "VBUS" (id 1) (at -37.973 184.5838 0)
+      (effects (font (size 1.27 1.27)) (justify right))
+    )
+    (property "Footprint" "" (id 2) (at -39.37 182.88 0)
+      (effects (font (size 1.27 1.27)) hide)
+    )
+    (property "Datasheet" "" (id 3) (at -39.37 182.88 0)
+      (effects (font (size 1.27 1.27)) hide)
+    )
+    (pin "1")
   )
   (symbol (lib_id "power:GND") (at 76.2 58.42 0) (unit 1)
@@
     )
     (property "Datasheet" "" (id 3) (at 35.56 115.57 0)
+      (effects (font (size 1.27 1.27)) hide)
+    )
+    (pin "1")
+  )
+  (symbol (lib_id "power:PWR_FLAG") (at -29.21 182.88 0) (unit 1)
+    (in_bom yes) (on_board yes) (fields_autoplaced)
+    (property "Reference" "#FLG?" (id 0) (at -29.21 180.975 0)
+      (effects (font (size 1.27 1.27)) hide)
+    )
+    (property "Value" "PWR_FLAG" (id 1) (at -29.21 179.3042 0))
+    (property "Footprint" "" (id 2) (at -29.21 182.88 0)
+      (effects (font (size 1.27 1.27)) hide)
+    )
+    (property "Datasheet" "~" (id 3) (at -29.21 182.88 0)
       (effects (font (size 1.27 1.27)) hide)
     )
@@
     (pin "1")
     (pin "2")
+  )
+  (symbol (lib_id "power:PWR_FLAG") (at -39.37 182.88 0) (unit 1)
+    (in_bom yes) (on_board yes) (fields_autoplaced)
+    (property "Reference" "#FLG?" (id 0) (at -39.37 180.975 0)
+      (effects (font (size 1.27 1.27)) hide)
+    )
+    (property "Value" "PWR_FLAG" (id 1) (at -39.37 179.3042 0))
+    (property "Footprint" "" (id 2) (at -39.37 182.88 0)
+      (effects (font (size 1.27 1.27)) hide)
+    )
+    (property "Datasheet" "~" (id 3) (at -39.37 182.88 0)
+      (effects (font (size 1.27 1.27)) hide)
+    )
+    (pin "1")
   )
   (symbol (lib_id "My_Symbols:NFCModuleRC522") (at 168.91 55.88 0) (unit 1)
@@
     (pin "2")
   )
+  (symbol (lib_id "power:GND") (at -29.21 182.88 0) (unit 1)
+    (in_bom yes) (on_board yes) (fields_autoplaced)
+    (property "Reference" "#PWR?" (id 0) (at -29.21 189.23 0)
+      (effects (font (size 1.27 1.27)) hide)
+    )
+    (property "Value" "GND" (id 1) (at -29.21 187.3234 0))
+    (property "Footprint" "" (id 2) (at -29.21 182.88 0)
+      (effects (font (size 1.27 1.27)) hide)
+    )
+    (property "Datasheet" "" (id 3) (at -29.21 182.88 0)
+      (effects (font (size 1.27 1.27)) hide)
+    )
+    (pin "1")
+  )
   (symbol (lib_id "power:+3V3") (at 166.37 100.33 0) (unit 1)
     (in_bom yes) (on_board yes) (fields_autoplaced)
@@
   )
   (symbol_instances
+    (path "/43cc4efe-4f0b-451c-a04f-d9b691a70901"
+      (reference "#FLG?") (unit 1) (value "PWR_FLAG") (footprint "")
+    )
+    (path "/47257b1f-54ef-46c8-8f75-e68befc97396"
+      (reference "#FLG?") (unit 1) (value "PWR_FLAG") (footprint "")
+    )
+    (path "/c94e449b-b7c1-4e28-96dd-4a2137a0f708/702bad6a-d69b-4a6f-8b7a-fde40c1a347a"
+      (reference "#FLG?") (unit 1) (value "PWR_FLAG") (footprint "")
+    )
     (path "/6c1df1a7-a844-4808-9980-ebbffa652994"
       (reference "#PWR01") (unit 1) (value "VBUS") (footprint "")
@@
       (reference "#PWR0103") (unit 1) (value "+3V3") (footprint "")
     )
+    (path "/164be65e-2346-4de9-bf84-11f530f17015"
+      (reference "#PWR?") (unit 1) (value "VBUS") (footprint "")
+    )
+    (path "/caff6b2c-24c7-43a1-af8f-a1f13e3b9e23"
+      (reference "#PWR?") (unit 1) (value "GND") (footprint "")
+    )
     (path "/8bd10394-54dc-41a7-a550-9a29b6db628e"
