File: pcb/NFC2USB.kicad_sch (KiCad schematic)
At the start: 12 parts, among them J1 USB_C_Receptacle_USB2.0, U1 NFCModuleRC522, U2 AMS1117-3.3

Commit message: feat: change from ESP32 to RP2040
Changing the Microcontroller to RP2040 because of price, availability and ease of use
Parts:
- added SW2: MODE, Button_Switch_SMD:SW_SPDT_PCM12, symbol Switch:SW_SPDT
- J1: value USB_C_Receptacle_USB2.0 -> USB_C_USB2.0
Connections:
- net +3V3: now also SW2.3 (C); no longer D1.2 (A), D2.2 (A)
- net GND: now also R3.2, R4.2, SW2.1 (A)
- net LED_ACT: now also D2.2 (A); no longer R4.2
- net LED_RDY: now also D1.2 (A); no longer R3.2
- new net MODE: SW2.2 (B)
Other:
- removed sheet ESP32-S2
- added sheet RP2040 (rp2040.kicad_sch)
- moved on the sheet: D1, D2, R3, R4
