File: pcb/NFC2USB.kicad_pcb (KiCad board)
At the start: 4 copper layers, 39 x 40 mm, 44 parts, among them J1 USB_C_Receptacle_USB2.0, J2 UART, U1 NFCModuleRC522, U2 AMS1117-3.3, U3 ESP32-S2FH4, Y1 X322540MPB4SI

Commit message: style: (re)move overlapping silkscreen objects
Parts:
- removed G***: LOGO, My_Footprints:CutieMark5mmInverted
Connections:
- net /ESP32-S2/U0RXD renamed /ESP32-S2/RX
