File: pcb/NFC2USB.kicad_pcb (KiCad board)
At the start: 4 copper layers, 39 x 40 mm, 43 parts, among them J1 USB_C_Receptacle_USB2.0, J2 UART, U1 NFCModuleRC522, U2 AMS1117-3.3, U3 ESP32-S2FH4, Y1 X322540MPB4SI

Commit message: feat: change from ESP32 to RP2040
Changing the Microcontroller to RP2040 because of price, availability and ease of use
Parts:
- removed C10: 10u, Capacitor_SMD:C_0603_1608Metric
- removed J2: UART, Connector_PinSocket_2.54mm:PinSocket_1x05_P2.54mm_Vertical
- removed L1: 2nH, Inductor_SMD:L_0402_1005Metric
- removed R10: 0R, Resistor_SMD:R_0402_1005Metric
- removed R5: 10k, Resistor_SMD:R_0402_1005Metric
- added C18: 15p, Capacitor_SMD:C_0402_1005Metric, F.Cu at (115.0, 78.5)
- added C19: 15p, Capacitor_SMD:C_0402_1005Metric, F.Cu at (109.5, 79.0)
- added G***: LOGO, My_Footprints:CutieMark5mmInverted, B.Cu at (111.8, 65.0)
- added SW1: BOOTSEL, Button_Switch_SMD:SW_SPST_TL3342, F.Cu at (110.0, 53.2)
- added SW2: MODE, Button_Switch_SMD:SW_SPDT_PCM12, F.Cu at (123.0, 70.0)
- added U4: RP2040, Package_DFN_QFN:QFN-56-1EP_7x7mm_P0.4mm_EP3.2x3.2mm, F.Cu at (112.5, 70.0)
- C11, C4: value 1u -> 100n
- C14: value 100n -> 1u
- C16: value 22p -> 1u
- C17, C5, C6: value 22p -> 100n
- J1: value USB_C_Receptacle_USB2.0 -> USB_C_USB2.0
- R6: value 470R -> 27R
- R8: value 27R -> 1k
- R9: value 10k -> 1k
- U3: value ESP32-S2FH4 -> W25Q32JVSS; footprint Package_DFN_QFN:QFN-56-1EP_7x7mm_P0.4mm_EP5.6x5.6mm -> Package_SO:SOIC-8_5.23x5.23mm_P1.27mm
- Y1: value X322540MPB4SI -> 12MHz
- moved R8 21.2 mm to (105.0, 55.2)
- moved Y1 19.8 mm to (112.2, 78.8)
- moved C16 17.8 mm to (116.0, 57.8), turned to 90 degrees
- moved C17 17.8 mm to (115.0, 57.8), turned to 90 degrees
- moved C4 13.3 mm to (113.5, 75.5), turned to 90 degrees
- moved C11 12.9 mm to (117.2, 72.0)
- moved C13 11.5 mm to (114.5, 75.5)
- moved R6 10.6 mm to (115.8, 63.7), turned to 180 degrees
- moved R1 9.87 mm to (116.2, 85.8), turned to 180 degrees
- moved C7 9.85 mm to (107.8, 66.8), turned to -90 degrees
- moved C15 9.71 mm to (117.8, 65.2), turned to 180 degrees
- moved C5 9.55 mm to (117.8, 66.2), turned to 180 degrees
- moved R7 9.29 mm to (115.8, 64.7), turned to 180 degrees
- moved U3 9.28 mm to (109.8, 59.2)
- moved C8 9.25 mm to (107.8, 72.0), turned to 90 degrees
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Connections:
- C11 pad 1: +3V3 -> GND
- C11 pad 2: GND -> +3V3
- C12 pad 1: +3V3 -> GND
- C12 pad 2: GND -> +1V1
- C13 pad 1: /ESP32-S2/VDD3P3 -> GND
- C13 pad 2: GND -> +1V1
- C14 pad 1: +3V3 -> GND
- C14 pad 2: GND -> +1V1
- C15 pad 1: +3V3 -> GND
- C15 pad 2: GND -> +3V3
- C16 pad 1: /USB_D- -> GND
- C16 pad 2: GND -> +3V3
- C17 pad 1: /USB_D+ -> GND
- C17 pad 2: GND -> +3V3
- C4 pad 1: /ESP32-S2/EN -> GND
- C4 pad 2: GND -> +3V3
- C5 pad 1: Net-(C5-Pad1) -> GND
- C5 pad 2: GND -> +3V3
- C6 pad 1: /ESP32-S2/XTAL_N -> GND
- C6 pad 2: GND -> +3V3
- C7 pad 1: +3V3 -> GND
- C7 pad 2: GND -> +3V3
- C8 pad 1: +3V3 -> GND
- C8 pad 2: GND -> +3V3
- C9 pad 1: +3V3 -> GND
- C9 pad 2: GND -> +3V3
- D1 pad 2: +3V3 -> /LED_RDY
- D2 pad 2: +3V3 -> /LED_ACT
- R3 pad 2: /LED_RDY -> GND
- R4 pad 2: /LED_ACT -> GND
- R6 pad 1: /ESP32-S2/U0TXD -> /USB_D+
- R6 pad 2: /ESP32-S2/TX -> /RP2040/USBD+
- R7 pad 1: /ESP32-S2/D+ -> /USB_D-
- R7 pad 2: /USB_D+ -> /RP2040/USBD-
- R8 pad 1: /ESP32-S2/D- -> /RP2040/BOOTSEL
- R8 pad 2: /USB_D- -> /RP2040/QSPI_SS
- R9 pad 1: /ESP32-S2/GPIO18 -> /RP2040/XR
- R9 pad 2: +3V3 -> /RP2040/XOUT
- U3 pad 1: +3V3 -> /RP2040/QSPI_SS
- U3 pad 2: unconnected-(U3-Pad2) -> /RP2040/QSPI_SD1
- U3 pad 3: /ESP32-S2/VDD3P3 -> /RP2040/QSPI_SD2
- U3 pad 4: /ESP32-S2/VDD3P3 -> GND
- U3 pad 5: /ESP32-S2/GPIO0 -> /RP2040/QSPI_SD0
- U3 pad 6: /NFC_Reset -> /RP2040/QSPI_SCLK
- U3 pad 7: /NFC_IRQ -> /RP2040/QSPI_SD3
- U3 pad 8: /NFC_MISO -> +3V3
- Y1 pad 1: Net-(C5-Pad1) -> /RP2040/XIN
- Y1 pad 3: /ESP32-S2/XTAL_N -> /RP2040/XR
Routing:
- net /ESP32-S2/GPIO0: track 18.1 -> 0.00 mm, vias 2 -> 0
- net /USB_D+: track 14.6 -> 31.2 mm
- net /USB_D-: track 14.2 -> 30.5 mm, vias 0 -> 2
- net +1V1: track 0.00 -> 16.0 mm
- net /RP2040/QSPI_SS: track 0.00 -> 15.9 mm
- net /ESP32-S2/RX: track 15.6 -> 0.00 mm, vias 1 -> 0
- net /ESP32-S2/U0TXD: track 12.9 -> 0.00 mm, vias 2 -> 0
- net /RP2040/QSPI_SD1: track 0.00 -> 12.4 mm
- net /RP2040/QSPI_SD3: track 0.00 -> 11.5 mm, vias 0 -> 2
- net /RP2040/QSPI_SD2: track 0.00 -> 10.9 mm
- net /RP2040/QSPI_SCLK: track 0.00 -> 10.7 mm, vias 0 -> 2
- net /RP2040/QSPI_SD0: track 0.00 -> 10.3 mm, vias 0 -> 2
- net /ESP32-S2/XTAL_N: track 8.60 -> 0.00 mm
- net /RP2040/XIN: track 0.00 -> 8.60 mm
- net /RP2040/BOOTSEL: track 0.00 -> 8.32 mm
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Other:
- board text added: "BOOTSEL"
- board text added: "MODE"
- board text added: "RC522"
- board text removed: "IO0"
- board text removed: "RX"
- board text removed: "TX"
